File: hex-smd-challenge-v2.kicad_pcb (KiCad board)
At the start: 2 copper layers, 44 x 50 mm, 29 parts, among them CON1 AVR-ISP-6, IC1 IC1, P0 CONN_01X01, P1 CONN_01X01, P2 CONN_01X01, P3 CONN_01X01, P4 CONN_01X01

Commit message: add new version of design including v2 which went to fab
Parts:
- CON1: moved to B.Cu
- moved CON1 0.32 mm to (222.8, 86.2)
Routing:
- net Net-(CON1-Pad5): track 0.00 -> 42.3 mm, vias 0 -> 1
- net Net-(CON1-Pad4): track 24.6 -> 41.1 mm, vias 0 -> 1
- net Net-(CON1-Pad1): track 15.1 -> 28.1 mm, vias 0 -> 1
- net +BATT: track 12.0 -> 24.7 mm, vias 2 -> 3
- net Net-(CON1-Pad3): track 27.0 -> 37.0 mm, vias 0 -> 1
- net GND: track 26.7 -> 16.9 mm, vias 2 -> 4
Other:
- board text added: "OSHPark.com/ SMDChallenge"
- board text removed: "OSHPark.com/SMDChallenge"
